File: _autosave-usb to serial.kicad_pcb (KiCad board)
At the start: 2 copper layers, 9 parts, among them CON1 USB-MINI-B, P1 CONN_7, P2 CONN_1, P3 CONN_1, U1 CP2102

Commit message: added final files
Parts:
- added LOGO: , logo:LOGO (2), F.Cu at (32.2, 34.0)
- moved C2 70.4 mm to (40.9, 24.0)
- moved C3 70.4 mm to (50.7, 24.0)
- moved CON1 70.4 mm to (32.9, 29.6)
- moved D1 70.4 mm to (41.0, 33.9)
- moved P2 70.4 mm to (45.5, 22.5)
- moved R1 70.4 mm to (50.7, 33.9)
- moved P1 70.4 mm to (56.8, 29.6)
- moved P3 70.4 mm to (45.6, 36.7)
- moved U1 70.4 mm to (45.6, 29.6)
Routing:
- net GND: track 71.6 -> 74.6 mm
Other:
- board outline added: 30 x 20 mm
- board text added: "ExploreEmbedded.com"
