File: usb to serial.kicad_pcb (KiCad board)
At the start: 2 copper layers, 9 parts, among them CON1 USB-MINI-B, P1 CONN_7, P2 CONN_1, P3 CONN_1, U1 CP2102

Commit message: added final files
Parts:
- added LOGO: , logo:LOGO (2), F.Cu at (32.2, 34.0)
- moved C2 70.4 mm to (40.9, 24.0)
- moved C3 70.4 mm to (50.7, 24.0)
- moved CON1 70.4 mm to (32.9, 29.6)
- moved D1 70.4 mm to (41.0, 33.9)
- moved P2 70.4 mm to (45.5, 22.5)
- moved R1 70.4 mm to (50.7, 33.9)
- moved P1 70.4 mm to (56.8, 29.6)
- moved P3 70.4 mm to (45.6, 36.7)
- moved U1 70.4 mm to (45.6, 29.6)
Routing:
- net GND: track 71.6 -> 74.6 mm
Other:
- board outline added: 30 x 20 mm
- board text added: "ExploreEmbedded.com"

Commit message: Fritzing part added
Routing:
- added copper zone on F.Cu, net /VCC
- added copper zone on B.Cu, net GND
Changed lines of the file:
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@@
     (links 24)
     (no_connects 0)
-    (area 28.309499 19.309499 58.690501 39.690501)
+    (area 23.096477 18.4 62.553429 40.436)
     (thickness 1.6002)
     (drawings 26)
@@
     (mod_text_size 1.524 1.524)
     (mod_text_width 0.3048)
-    (pad_size 1.8 0.4)
-    (pad_drill 0)
+    (pad_size 1.905 2.286)
+    (pad_drill 0.8128)
     (pad_to_mask_clearance 0.254)
     (aux_axis_origin 0 0)
     (visible_elements 7FFFFFFF)
     (pcbplotparams
-      (layerselection 0x00030_80000001)
-      (usegerberextensions true)
+      (layerselection 0x00020_00000000)
+      (usegerberextensions false)
       (excludeedgelayer false)
       (linewidth 0.150000)
@@
       (padsonsilk false)
       (subtractmaskfromsilk false)
-      (outputformat 1)
+      (outputformat 5)
       (mirror false)
-      (drillshape 1)
+      (drillshape 0)
       (scaleselection 1)
       (outputdirectory gerber/))
@@
     (pad 5 smd rect (at 1.2991 -1.8) (size 1.8 0.4) (layers Front F.Paste F.Mask)
       (net 9 GND))
-    (pad 6 thru_hole oval (at -2.5009 -1.56254) (size 0.95 1.25) (drill oval 0.55 0.85) (layers *.Cu *.Mask F.SilkS)
+    (pad 6 thru_hole oval (at -2.5009 -1.56254) (size 1.2 1.3) (drill oval 0.85) (layers *.Cu *.Mask F.SilkS)
       (net 9 GND))
-    (pad 6 thru_hole oval (at 2.4991 -1.56254) (size 0.95 1.25) (drill oval 0.55 0.85) (layers *.Cu *.Mask F.SilkS)
+    (pad 6 thru_hole oval (at 2.4991 -1.56254) (size 1.2 1.3) (drill oval 0.85) (layers *.Cu *.Mask F.SilkS)
       (net 9 GND))
     (pad 6 smd rect (at -4.6 1.1) (size 1.55 2.5) (layers Front F.Paste F.Mask)
@@
   (segment (start 49.291 35.343) (end 50.149185 34.484815) (width 0.508) (layer Front) (net 11))
   (segment (start 41.574815 34.484815) (end 42.306 35.216) (width 0.3048) (layer Front) (net 11))
+  (zone (net 9) (net_name GND) (layer Back) (hatch edge 0.508)
+    (connect_pads (clearance 0.508))
+    (min_thickness 0.254)
+    (fill yes (arc_segments 16) (thermal_gap 0.508) (thermal_bridge_width 0.508))
+    (polygon
+      (pts
+        (xy 58 39) (xy 29 39) (xy 29 20) (xy 58 20)
+      )
+    )
+  )
+  (zone (net 8) (net_name /VCC) (layer Front) (hatch edge 0.508)
+    (connect_pads (clearance 0.508))
+    (min_thickness 0.254)
+    (fill yes (arc_segments 16) (thermal_gap 0.508) (thermal_bridge_width 0.508))
+    (polygon
+      (pts
+        (xy 58 39) (xy 29 39) (xy 29 20) (xy 58 20)
+      )
+    )
+  )
 )
